Commit message: WS hardware interface works but th esp32 connection is unstable. Try to put the webserver on dedicated core

File: ros_ws/src/sb_robot/description/ros2_control.xacro (robot description, xacro)
@@ -1,5 +1,4 @@
 <?xml version="1.0"?>
 <robot xmlns:xacro="http://www.ros.org/wiki/xacro">
-    <!-- <xacro:unless value="$(arg sim_mode)"> -->
         <ros2_control name="RealRobot" type="system">
             <hardware>
@@ -9,6 +8,5 @@
                 <param name="left_wheel_letter">B</param>
                 <param name="right_wheel_letter">A</param>
-                <!-- <param name="lidar_name">laser_joint</param> -->
-                <param name="device_addr">ws://192.168.1.77:80/ws</param>
+                <param name="device_address">ws://192.168.1.77:80/ws</param>
                 <param name="device_token">your_secret_token</param>
                 <param name="timeout_ms">1000</param>
@@ -30,54 +28,4 @@
                 <state_interface name="velocity"/>
             </joint>
-            <!-- TEST rotating lidar-->
-            <!-- <joint name="laser_joint">
-                <command_interface name="velocity">
-                    <param name="min">-10</param>
-                    <param name="max">10</param>
-                </command_interface>
-                <state_interface name="position"/>
-                <state_interface name="velocity"/>
-            </joint> -->
-            <!-- TEST rotating lidar-->
         </ros2_control>
-    <!-- </xacro:unless> -->
-    <!-- <xacro:if value="$(arg sim_mode)">
-        <ros2_control name="GazeboSystem" type="system">
-            <hardware>
-                <plugin>gazebo_ros2_control/GazeboSystem</plugin>
-            </hardware>
-            <joint name="left_wheel_joint">
-                <command_interface name="velocity">
-                    <param name="min">-10</param>
-                    <param name="max">10</param>
-                </command_interface>
-                <state_interface name="velocity"/>
-                <state_interface name="position"/>
-            </joint>
-            <joint name="right_wheel_joint">
-                <command_interface name="velocity">
-                    <param name="min">-10</param>
-                    <param name="max">10</param>
-                </command_interface>
-                <state_interface name="velocity"/>
-                <state_interface name="position"/>
-            </joint> -->
-            <!-- TEST rotating lidar-->
-            <!-- <joint name="laser_joint">
-                <command_interface name="velocity">
-                    <param name="min">-10</param>
-                    <param name="max">10</param>
-                </command_interface>
-                <state_interface name="position"/>
-                <state_interface name="velocity"/>
-            </joint> -->
-            <!-- TEST rotating lidar-->
-        <!-- </ros2_control> -->
-    <!-- </xacro:if>
-    <gazebo>
-        <plugin name="gazebo_ros2_control" filename="libgazebo_ros2_control.so">
-            <parameters>$(find boxbot_description)/config/my_controllers.yaml</parameters>
-            <parameters>$(find boxbot_description)/config/gaz_ros2_ctl_use_sim.yaml</parameters>
-        </plugin>
-    </gazebo> -->
 </robot>
