Commit message: pitch published to joint_states. PIDs work incorrectly

File: ros_ws/src/sb_robot/description/robot_core.xacro (robot description, xacro)
@@ -38,5 +38,5 @@
 </link>
 <!-- CHASSIS LINK-->
-<joint
+  <!-- <joint
     name="chassis_joint"
     type="fixed">
@@ -50,4 +50,19 @@
     <axis
       xyz="0 0 0" />
+  </joint> -->
+  <joint
+    name="chassis_joint"
+    type="revolute">
+    <origin
+      xyz="0 0 0"
+      rpy="0 0 0" />
+    <parent
+      link="base_link" />
+    <child
+      link="chassis_link" />
+    <axis
+      xyz="0 1 0" />
+    <dynamics damping="0.5" friction="0.1" />
+    <limit effort="1000.0" lower="-1.57" upper="1.57" velocity="10.0"/>
   </joint>
   <link
